File: thinkpad-teensy-keyboard/thinkpad-teensy-keyboard/thinkpad-teensy-keyboard.kicad_pcb (KiCad board)
At the start: 2 copper layers, 10 parts, among them J2 WM6787CT-ND, J3 3, Q1 220mA/50V/3.5Ω, Q2 220mA/50V/3.5Ω, U1 Teensy4.1

Commit message: Generated Gerbers
Parts:
- removed J3: 3, Library:1X01
- added GOLD_ORB_SM1: OSHWLOGOLOGO5MM, Library:OSHW_5MM, F.Cu at (120.4, 65.6)
- J2: moved to B.Cu
- U1: footprint teensy:Teensy41 -> teensy:Teensy41_ignore_ethernet_no_silk
- moved U1 32.1 mm to (120.0, 78.2)
- moved R5 23.7 mm to (119.0, 56.3), turned to 180 degrees
- moved Q1 22.4 mm to (122.3, 53.3), turned to 180 degrees
- moved Q2 20.2 mm to (118.5, 53.3), turned to 180 degrees
- moved R4 18.8 mm to (123.3, 56.3)
- moved J2 14.7 mm to (120.0, 77.2)
- moved R3 9.09 mm to (122.3, 49.7), turned to 90 degrees
- moved R2 8.59 mm to (118.5, 49.7), turned to 90 degrees
- moved C1 7.67 mm to (115.3, 49.0), turned to 180 degrees
Connections:
- J2 pad P$11: Net-(J2-PadP$11) -> Net-(U1-Pad42)
- J2 pad P$13: Net-(J2-PadP$13) -> Net-(U1-Pad43)
- J2 pad P$15: Net-(J2-PadP$15) -> Net-(U1-Pad44)
- J2 pad P$17: Net-(J2-PadP$17) -> Net-(U1-Pad45)
- J2 pad P$20: Net-(J2-PadP$20) -> Net-(U1-Pad12)
- J2 pad P$22: Net-(J2-PadP$22) -> Net-(U1-Pad11)
- J2 pad P$24: Net-(J2-PadP$24) -> Net-(U1-Pad10)
- J2 pad P$26: Net-(J2-PadP$26) -> Net-(U1-Pad9)
- J2 pad P$28: Net-(J2-PadP$28) -> Net-(U1-Pad8)
- J2 pad P$3: Net-(J2-PadP$3) -> Net-(U1-Pad38)
- J2 pad P$30: Net-(J2-PadP$30) -> Net-(U1-Pad7)
- J2 pad P$32: Net-(J2-PadP$32) -> Net-(U1-Pad6)
- J2 pad P$36: Net-(J2-PadP$36) -> Net-(U1-Pad5)
- J2 pad P$4: Net-(J2-PadP$4) -> Net-(U1-Pad32)
- J2 pad P$40: Net-(J2-PadP$40) -> Net-(U1-Pad4)
- J2 pad P$5: Net-(J2-PadP$5) -> Net-(U1-Pad39)
- J2 pad P$7: Net-(J2-PadP$7) -> Net-(U1-Pad40)
- J2 pad P$9: Net-(J2-PadP$9) -> Net-(U1-Pad41)
- Q1 pad 2: Net-(J2-PadP$39) -> Net-(Q1-Pad2)
- R3 pad 1: Net-(J2-PadP$39) -> Net-(Q1-Pad2)
- U1 pad 10: Net-(J2-PadP$13) -> Net-(U1-Pad10)
- U1 pad 11: Net-(J2-PadP$5) -> Net-(U1-Pad11)
- U1 pad 12: Net-(J2-PadP$36) -> Net-(U1-Pad12)
- U1 pad 13: Net-(J2-PadP$1) -> Net-(J2-PadP$18)
- U1 pad 14: unconnected-(U1-Pad14) -> Net-(J2-PadP$16)
- U1 pad 16: unconnected-(U1-Pad16) -> Net-(J2-PadP$14)
- U1 pad 17: unconnected-(U1-Pad17) -> Net-(J2-PadP$12)
- U1 pad 18: unconnected-(U1-Pad18) -> Net-(J2-PadP$10)
- U1 pad 28: Net-(J2-PadP$40) -> unconnected-(U1-Pad28)
- U1 pad 29: Net-(J2-PadP$30) -> unconnected-(U1-Pad29)
- U1 pad 3: Net-(J2-PadP$39) -> Net-(Q1-Pad2)
- U1 pad 30: Net-(J2-PadP$26) -> unconnected-(U1-Pad30)
- U1 pad 31: Net-(J2-PadP$32) -> Net-(J2-PadP$19)
- U1 pad 32: Net-(J2-PadP$28) -> Net-(U1-Pad32)
- U1 pad 33: Net-(J2-PadP$24) -> Net-(J2-PadP$2)
- U1 pad 35: Net-(J2-PadP$16) -> Net-(J2-PadP$6)
- U1 pad 36: Net-(J2-PadP$20) -> Net-(J2-PadP$8)
- U1 pad 37: Net-(J2-PadP$6) -> Net-(J2-PadP$1)
- U1 pad 38: Net-(J2-PadP$12) -> Net-(U1-Pad38)
- U1 pad 39: Net-(J2-PadP$8) -> Net-(U1-Pad39)
- U1 pad 4: Net-(J2-PadP$17) -> Net-(U1-Pad4)
- U1 pad 40: Net-(J2-PadP$4) -> Net-(U1-Pad40)
- U1 pad 41: Net-(J2-PadP$2) -> Net-(U1-Pad41)
- U1 pad 42: Net-(J2-PadP$10) -> Net-(U1-Pad42)
- U1 pad 43: Net-(J2-PadP$14) -> Net-(U1-Pad43)
- U1 pad 44: Net-(J2-PadP$18) -> Net-(U1-Pad44)
- U1 pad 45: Net-(J2-PadP$22) -> Net-(U1-Pad45)
- U1 pad 5: Net-(J2-PadP$15) -> Net-(U1-Pad5)
- U1 pad 6: Net-(J2-PadP$3) -> Net-(U1-Pad6)
- U1 pad 7: Net-(J2-PadP$11) -> Net-(U1-Pad7)
- U1 pad 8: Net-(J2-PadP$7) -> Net-(U1-Pad8)
- U1 pad 9: Net-(J2-PadP$9) -> Net-(U1-Pad9)
Routing:
- net GND: track 0.00 -> 76.8 mm, vias 0 -> 1
- net +3V3: track 0.00 -> 59.6 mm, vias 0 -> 1
- net +5V: track 0.00 -> 44.1 mm, vias 0 -> 1
- net Net-(U1-Pad4): track 0.00 -> 25.3 mm, vias 0 -> 1
- net Net-(U1-Pad45): track 0.00 -> 23.9 mm
- net Net-(U1-Pad5): track 0.00 -> 23.5 mm, vias 0 -> 1
- net Net-(J2-PadP$37): track 0.00 -> 22.1 mm, vias 0 -> 1
- net Net-(U1-Pad44): track 0.00 -> 21.7 mm
- net Net-(U1-Pad6): track 0.00 -> 20.5 mm, vias 0 -> 1
- net Net-(J2-PadP$19): track 0.00 -> 19.7 mm, vias 0 -> 1
- net Net-(U1-Pad43): track 0.00 -> 19.7 mm
- net Net-(J2-PadP$39): track 0.00 -> 19.4 mm, vias 0 -> 1
- net Net-(U1-Pad32): track 0.00 -> 18.4 mm
- net Net-(U1-Pad42): track 0.00 -> 17.7 mm
- net Net-(J2-PadP$2): track 0.00 -> 16.0 mm
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Other:
- board outline added: 20 x 64 mm
- board text added: "Teensy 4.1 to Thinkpad X61 Keyboard adapter v1.0.0"
